File: schemata/vypočtová/vypočtová.kicad_sch (KiCad schematic)
At the start: 71 parts, among them SW1 SW_DPST_x2, SW2 SW_DPST_x2, SW3 SW_DPST_x2, SW4 SW_DPST_x2, SW5 SW_DPST_x2, SW6 SW_DPST_x2, SW7 SW_DPST_x2, SW8 SW_DPST_x2, U1 MCU, U10 UR, U11 UR, U12 Ucc, U13 Uf, U14 Ucc, U15 Uf, U16 UR, U17 Ucc, U18 Uf, U19 PLC, U2 PLC, U20 PLC, U21 MCU, U22 MCU, U23 MCU, U24 MCU, U25 PLC, U26 PLC, U27 PLC, U28 PLC, U29 PLC, U3 PLC, U30 PLC, U4 MCU, U5 MCU, U6 MCU, U7 Ucc, U8 UR, U9 Uf

Commit message: Sync from Obsidian (Práce s digitálními vstupy a výstupy a řízení (ovládání) na základě času): 2026-09-09 21:02 UTC — 0+ 6~ 0-
Connections:
- net at U6. (Vcc): now also D4.1 (K)
- net at U28. (GND): now also SW8.2 (B)
- net at U4. (Vcc): now also D3.2 (A)
